Commit message: working examples of the mpc

File: models/franka_description/robots/panda/franka2.urdf (robot description, URDF)
Before this commit: robot pandas, 41 links, 40 joints
Links:
- link panda2_leftfinger: mass 0.015 -> None; geometry collision sphere radius=0.03
- link panda2_rightfinger: geometry collision sphere radius=0.03
